File: LibreSolar_BMS48V.sch (EAGLE design)
At the start: 201 parts, among them IC1 BQ76940, K1 62000211622, K4 66200621122, K5 66201821122, Q10 DMN2004K, Q11 DMN2004K, Q12 DMN2004K, Q13 DMN2004K, Q14 DMN2004K, Q15 DMN2004K, Q16 DMN2004K, Q17 DMN2004K, Q18 DMN2004K, Q19 DMN2004K, Q4 BSS123, Q5 DMN2004K, Q6 DMN2004K, Q7 DMN2004K, Q8 DMN2004K, Q9 DMN2004K, U1 TJA1042T/3, U2 LMR16006X, U3 M24256-BW, U5 MIC5225, U6 STM32F072CB, X1 ABS25-32.768KHZ-6, Y1 8MHz

Commit message: several modifications made for details see README.md
Parts:
- removed CELLS: (no value), Wire_to_Board_Connectors_rev15d:66201821022
- removed K5: 66201821122, Wire_to_Board_Connectors_rev15d:66201821122
- added J1: (no value), Wire-to-Board (rev18a):66202021122
- added J2: (no value), Wire-to-Board (rev18a):66202021022
Connections:
- removed net !CAN_EN!: U6.PA15
- removed net CAN_STB: U1.STB
- new net C10.1: D17.A, J1.17, J2.17, Q15.S, R47.1
- new net C5.1: D12.A, J1.14, J2.14, Q10.S, R41.1
- new net CAN_STBB: U1.STB, U6.PA15
- net C0: now also J1.11, J2.11; no longer CELLS.10, K5.10
- net C1: now also J1.2, J2.2; no longer CELLS.2, K5.2
- net C10: now also J1.7, J2.7; no longer CELLS.15, D17.A, K5.15, Q15.S, R47.1
- net C11: now also J1.8, J2.8; no longer CELLS.7, K5.7
- net C12: now also J1.18, J2.18; no longer CELLS.16, K5.16
- net C13: now also J1.9, J2.9; no longer CELLS.8, K5.8
- net C14: now also J1.19, J2.19; no longer CELLS.17, K5.17
- net C15: now also J1.10, J2.10; no longer CELLS.9, K5.9
- net C2: now also J1.12, J2.12; no longer CELLS.11, K5.11
- net C3: now also J1.3, J2.3; no longer CELLS.3, K5.3
- net C4: now also J1.13, J2.13; no longer CELLS.12, K5.12
- net C5: now also J1.4, J2.4; no longer CELLS.4, D12.A, K5.4, Q10.S, R41.1
- net C6: now also J1.5, J2.5; no longer CELLS.13, K5.13
- net C7: now also J1.15, J2.15; no longer CELLS.5, K5.5
- net C8: now also J1.6, J2.6; no longer CELLS.14, K5.14
- net C9: now also J1.16, J2.16; no longer CELLS.6, K5.6
- net GND: now also J1.1, J2.1; no longer CELLS.1, K5.1
- net PWR: now also J1.20, J2.20; no longer CELLS.18, K5.18
